Commit message: Add feet links to urdf

File: src/environment/urdf/robot-simple.urdf (robot description, URDF)
Before this commit: robot bipedal, 13 links, 12 joints
Links:
- added link back_left_foot, mass 0.1; collision sphere radius=0.1; visual sphere radius=0.1
- added link back_right_foot, mass 0.1; collision sphere radius=0.1; visual sphere radius=0.1
- added link left_foot, mass 0.1; collision sphere radius=0.1; visual sphere radius=0.1
- added link right_foot, mass 0.1; collision sphere radius=0.1; visual sphere radius=0.1
Joints:
- added joint back_left_leg_bottom_back_left_foot: type fixed, parent back_left_leg_bottom, child back_left_foot, origin xyz=0 0 0, axis 1 0 0
- added joint back_right_leg_bottom_back_right_foot: type fixed, parent back_right_leg_bottom, child back_right_foot, origin xyz=0 0 0, axis 1 0 0
- added joint left_leg_bottom_left_foot: type fixed, parent left_leg_bottom, child left_foot, origin xyz=0 0 0, axis 1 0 0
- added joint right_leg_bottom_right_foot: type fixed, parent right_leg_bottom, child right_foot, origin xyz=0 0 0, axis 1 0 0

Commit message: Increase mass

File: src/environment/urdf/robot-simple.urdf (robot description, URDF)
Before this commit: robot bipedal, 17 links, 16 joints
Links:
- link back_left_leg_bottom: mass 3 -> 5
- link back_left_leg_top: mass 7 -> 20
- link back_left_shoulder: mass 7 -> 10
- link back_right_leg_bottom: mass 3 -> 5
- link back_right_leg_top: mass 7 -> 20
- link back_right_shoulder: mass 7 -> 10
- link core: mass 30 -> 50
- link left_leg_bottom: mass 3 -> 5
- link left_leg_top: mass 7 -> 20
- link left_shoulder: mass 7 -> 10
- link right_leg_bottom: mass 3 -> 5
- link right_leg_top: mass 7 -> 20
- link right_shoulder: mass 7 -> 10

Commit message: change params

File: src/environment/urdf/robot-simple.urdf (robot description, URDF)
Before this commit: robot bipedal, 17 links, 16 joints
Joints:
- joint back_left_leg_top_back_left_leg_bottom: limit lower=-0.785398 upper=0.785398 effort=100 velocity=100 -> lower=-0.785398 upper=0.785398 effort=1000 velocity=1000
- joint back_left_shoulder_back_right_leg_top: limit lower=-0.785398 upper=0.785398 effort=100 velocity=100 -> lower=-0.785398 upper=0.785398 effort=1000 velocity=1000
- joint back_right_leg_top_back_right_leg_bottom: limit lower=-0.785398 upper=0.785398 effort=100 velocity=100 -> lower=-0.785398 upper=0.785398 effort=1000 velocity=1000
- joint back_right_shoulder_back_right_leg_top: limit lower=-0.785398 upper=0.785398 effort=100 velocity=100 -> lower=-0.785398 upper=0.785398 effort=1000 velocity=1000
- joint core_back_left_shoulder: limit lower=-0.785398 upper=0.785398 effort=100 velocity=100 -> lower=-0.785398 upper=0.785398 effort=1000 velocity=1000
- joint core_back_right_shoulder: limit lower=-0.785398 upper=0.785398 effort=100 velocity=100 -> lower=-0.785398 upper=0.785398 effort=1000 velocity=1000
- joint core_left_shoulder: limit lower=-0.785398 upper=0.785398 effort=100 velocity=100 -> lower=-0.785398 upper=0.785398 effort=1000 velocity=1000
- joint core_right_shoulder: limit lower=-0.785398 upper=0.785398 effort=100 velocity=100 -> lower=-0.785398 upper=0.785398 effort=1000 velocity=1000
- joint left_leg_top_left_leg_bottom: limit lower=-0.785398 upper=0.785398 effort=100 velocity=100 -> lower=-0.785398 upper=0.785398 effort=1000 velocity=1000
- joint left_shoulder_left_leg_top: limit lower=-0.785398 upper=0.785398 effort=100 velocity=100 -> lower=-0.785398 upper=0.785398 effort=1000 velocity=1000
- joint right_leg_top_right_leg_bottom: limit lower=-0.785398 upper=0.785398 effort=100 velocity=100 -> lower=-0.785398 upper=0.785398 effort=1000 velocity=1000
- joint right_shoulder_right_leg_top: limit lower=-0.785398 upper=0.785398 effort=100 velocity=100 -> lower=-0.785398 upper=0.785398 effort=1000 velocity=1000

Commit message: Change urdf file masses

File: src/environment/urdf/robot-simple.urdf (robot description, URDF)
Before this commit: robot bipedal, 17 links, 16 joints
Links:
- link back_left_foot: mass 0.1 -> 0.05
- link back_left_leg_bottom: mass 5 -> 0.05
- link back_left_leg_top: mass 20 -> 0.25
- link back_left_shoulder: mass 10 -> 0.25
- link back_right_foot: mass 0.1 -> 0.05
- link back_right_leg_bottom: mass 5 -> 0.05
- link back_right_leg_top: mass 20 -> 0.25
- link back_right_shoulder: mass 10 -> 0.25
- link core: mass 50 -> 3.2
- link left_foot: mass 0.1 -> 0.05
- link left_leg_bottom: mass 5 -> 0.05
- link left_leg_top: mass 20 -> 0.05
- link left_shoulder: mass 10 -> 0.25
- link right_foot: mass 0.1 -> 0.05
- link right_leg_bottom: mass 5 -> 0.05
- link right_leg_top: mass 20 -> 0.25
- link right_shoulder: mass 10 -> 0.25
Joints:
- joint back_left_leg_top_back_left_leg_bottom: limit lower=-0.785398 upper=0.785398 effort=1000 velocity=1000 -> lower=-0.785398 upper=0.785398 effort=100 velocity=100
- joint back_left_shoulder_back_right_leg_top: limit lower=-0.785398 upper=0.785398 effort=1000 velocity=1000 -> lower=-0.785398 upper=0.785398 effort=100 velocity=100
- joint back_right_leg_top_back_right_leg_bottom: limit lower=-0.785398 upper=0.785398 effort=1000 velocity=1000 -> lower=-0.785398 upper=0.785398 effort=100 velocity=100
- joint back_right_shoulder_back_right_leg_top: limit lower=-0.785398 upper=0.785398 effort=1000 velocity=1000 -> lower=-0.785398 upper=0.785398 effort=100 velocity=100
- joint core_back_left_shoulder: limit lower=-0.785398 upper=0.785398 effort=1000 velocity=1000 -> lower=-0.785398 upper=0.785398 effort=100 velocity=100
- joint core_back_right_shoulder: limit lower=-0.785398 upper=0.785398 effort=1000 velocity=1000 -> lower=-0.785398 upper=0.785398 effort=100 velocity=100
- joint core_left_shoulder: limit lower=-0.785398 upper=0.785398 effort=1000 velocity=1000 -> lower=-0.785398 upper=0.785398 effort=100 velocity=100
- joint core_right_shoulder: limit lower=-0.785398 upper=0.785398 effort=1000 velocity=1000 -> lower=-0.785398 upper=0.785398 effort=100 velocity=100
- joint left_leg_top_left_leg_bottom: limit lower=-0.785398 upper=0.785398 effort=1000 velocity=1000 -> lower=-0.785398 upper=0.785398 effort=100 velocity=100
- joint left_shoulder_left_leg_top: limit lower=-0.785398 upper=0.785398 effort=1000 velocity=1000 -> lower=-0.785398 upper=0.785398 effort=100 velocity=100
- joint right_leg_top_right_leg_bottom: limit lower=-0.785398 upper=0.785398 effort=1000 velocity=1000 -> lower=-0.785398 upper=0.785398 effort=100 velocity=100
- joint right_shoulder_right_leg_top: limit lower=-0.785398 upper=0.785398 effort=1000 velocity=1000 -> lower=-0.785398 upper=0.785398 effort=100 velocity=100
